Commit message: work in progress

File: description/rover_model/urdf/stand_link.urdf.xacro (robot description, xacro)
@@ -130,5 +130,5 @@
     </link>
     <joint name="imu_joint" type="fixed">
-        <origin xyz="0.159347 0 0" rpy="0 0 0" />
+        <origin xyz="0.159347 0 0" rpy="0 -0.0174533 0" />
         <!-- The x-pos is same as it's actual position on the stand, but z-pos same as base_link
              x: imu_x_dist_to_stand + chassis_to_stand_link_x_dist -->

Commit message: updated the urdf file to get a better relative position

File: description/rover_model/urdf/stand_link.urdf.xacro (robot description, xacro)
@@ -130,5 +130,5 @@
     </link>
     <joint name="imu_joint" type="fixed">
-        <origin xyz="0.159347 0 0" rpy="0 -0.0174533 0" />
+        <origin xyz="0.159347 0 0" rpy="0 -0.0349 0" />
         <!-- The x-pos is same as it's actual position on the stand, but z-pos same as base_link
              x: imu_x_dist_to_stand + chassis_to_stand_link_x_dist -->
