Commit message: Implemented+tested cartographer SLAM - modified urdf so imu link to be at same height as base_link

File: description/rover_model/urdf/constants.xacro (robot description, xacro)
@@ -6,7 +6,8 @@
     <xacro:property name="base_height" value="0.01"/> -->
     <!-- Chassis -->
-    <!-- <xacro:property name="chassis_to_base_link_dist" value="0.501747"/>
-    <xacro:property name="chassis_to_stand_link_dist" value="0.428526"/>
-    <xacro:property name="chassis_link_mass" value="36.95"/> -->
+    <xacro:property name="chassis_to_base_link_dist" value="0.34041"/>
+    <xacro:property name="chassis_to_stand_link_z_dist" value="0.26861"/>
+    <xacro:property name="chassis_to_stand_link_x_dist" value="0.178"/>
+    <xacro:property name="chassis_link_mass" value="36.95"/>
     <!-- Stand -->
     <!-- <xacro:property name="stand_length" value="0.412"/>
@@ -106,3 +107,6 @@
     <xacro:property name="imu_topic" value="imu/data"/>
     <xacro:property name="imu_update_rate" value="128.0"/>
+    <xacro:property name="imu_x_dist_to_stand" value="-0.018653"/>
+    <xacro:property name="imu_y_dist_to_stand" value="-0.001408"/>
+    <xacro:property name="imu_z_dist_to_stand" value="0.009525"/>
 </robot>

File: description/rover_model/urdf/espresso.urdf.xacro (robot description, xacro)
@@ -40,5 +40,5 @@
 	</link>
 	<joint name="chassis_joint" type="fixed">
-		<origin xyz="-0.004064 0 0.34041" rpy="0 0 0" />
+		<origin xyz="0 0 0.34041" rpy="0 0 0" />
 		<parent link="base_link" />
 		<child link="chassis_link" />

File: description/rover_model/urdf/plugins.gazebo.xacro (robot description, xacro)
@@ -26,5 +26,5 @@
         </plugin>
     </gazebo>
-    <!-- lets all the transmission tags be read -->
+    <!-- Lets all the transmission tags be read -->
     <gazebo>
         <plugin name="gazebo_ros_control" filename="libgazebo_ros_control.so"/>

File: description/rover_model/urdf/stand_link.urdf.xacro (robot description, xacro)
@@ -98,4 +98,5 @@
     </joint>
     <!-- IMU -->
+    <!-- Due to the requirements of cartographer, the imu_link frame is located on same height as base_link, but the model is located on top of the stand -->
     <link name="imu_link">
         <inertial>
@@ -111,5 +112,7 @@
         </inertial>
         <visual>
-            <origin xyz="0 0 0" rpy="0 0 0" />
+            <origin xyz="0 0 0.61854" rpy="0 0 0" /> <!-- Physical imu located on stand -->
+            <!-- z-pos of visual model moved back up to stand height
+                 z: imu_z_dist_to_stand + chassis_to_stand_link_z_dist + chassis_to_base_link_dist} -->
             <geometry>
                 <mesh filename="package://description/rover_model/meshes/imu_link.STL" />
@@ -120,5 +123,5 @@
         </visual>
         <collision>
-            <origin xyz="0 0 0" rpy="0 0 0" />
+            <origin xyz="0 0 0.61854" rpy="0 0 0" />
             <geometry>
                 <mesh filename="package://description/rover_model/meshes/imu_link.STL" />
@@ -127,6 +130,8 @@
     </link>
     <joint name="imu_joint" type="fixed">
-        <origin xyz="-0.018653 -0.001408 0.009525" rpy="0 0 0" />
-        <parent link="stand_link" />
+        <origin xyz="0.159347 0 0" rpy="0 0 0" />
+        <!-- The x-pos is same as it's actual position on the stand, but z-pos same as base_link
+             x: imu_x_dist_to_stand + chassis_to_stand_link_x_dist -->
+        <parent link="base_link" /> <!-- The frame origin is centered on base_link -->
         <child link="imu_link" />
         <axis xyz="0 0 0" />

Commit message: Changed lidar simulation range to 180 degrees to prevent self-collision (not solved for irl yet)

File: description/rover_model/urdf/constants.xacro (robot description, xacro)
@@ -49,5 +49,5 @@
     <xacro:property name="laser_horizontal_resolution" value="1"/>
     <xacro:property name="laser_horizontal_samples" value="1080"/>
-    <xacro:property name="laser_field_of_view" value="270"/>
+    <xacro:property name="laser_field_of_view" value="180"/>
     <xacro:property name="laser_horizontal_min_angle" value="${-0.5*laser_field_of_view*pi/180}"/>
     <xacro:property name="laser_horizontal_max_angle" value="${0.5*laser_field_of_view*pi/180}"/>

Commit message: Updated filter_lidar to reflect changes in caff.

File: description/rover_model/urdf/constants.xacro (robot description, xacro)
@@ -49,9 +49,9 @@
     <xacro:property name="laser_horizontal_resolution" value="1"/>
     <xacro:property name="laser_horizontal_samples" value="1080"/>
-    <xacro:property name="laser_field_of_view" value="180"/>
+    <xacro:property name="laser_field_of_view" value="360"/>
     <xacro:property name="laser_horizontal_min_angle" value="${-0.5*laser_field_of_view*pi/180}"/>
     <xacro:property name="laser_horizontal_max_angle" value="${0.5*laser_field_of_view*pi/180}"/>
-    <xacro:property name="laser_range_min" value="0.06"/>
-    <xacro:property name="laser_range_max" value="4.095"/>
+    <xacro:property name="laser_range_min" value="0.15"/>
+    <xacro:property name="laser_range_max" value="8"/>
     <xacro:property name="laser_resolution_angle" value="0.36"/>
     <xacro:property name="laser_range_resolution" value="${laser_resolution_angle*pi/180}"/>

Commit message: Adjusted zed urdf to match irl

File: description/rover_model/urdf/constants.xacro (robot description, xacro)
@@ -90,5 +90,5 @@
     <!--ZED CAMERA JOINT PARAMETERS-->
     <xacro:property name="ZED_camera_to_top_plate_x" value="${(stand_width / 2.0)-0.01}"/>
-    <xacro:property name="ZED_camera_to_top_plate_z" value="0.065"/>
+    <xacro:property name="ZED_camera_to_top_plate_z" value="0.10098"/>
     <!-- Garmin GPS -->
     <!-- NOTE: approx. as a cylinder, Garmin itself is similar to a hockey puck -->

File: description/rover_model/urdf/stand_link.urdf.xacro (robot description, xacro)
@@ -74,5 +74,5 @@
     </link>
     <joint name="zed_joint" type="fixed">
-        <origin xyz="0.044163 0 0.065" rpy="0 ${ZED_camera_pitch} 0" />
+        <origin xyz="0.044163 0 ${ZED_camera_to_top_plate_z}" rpy="0 ${ZED_camera_pitch} 0" />
         <parent link="stand_link" />
         <child link="zed_link" />

Commit message: Updates for running irl sensors

File: description/rover_model/urdf/constants.xacro (robot description, xacro)
@@ -71,5 +71,5 @@
     <xacro:property name="ZED_camera_length" value="0.175"/>
     <xacro:property name="ZED_stereo_offset" value="0.12"/>
-    <xacro:property name="ZED_camera_pitch" value="${20 * pi/180}"/>
+    <xacro:property name="ZED_camera_pitch" value="${30 * pi/180}"/>
     <!--<xacro:property name="ZED_camera_pitch" value="${50 * pi/180}"/>-->
     <!-- ZED image height/width corresponds to image size for 60Hz refresh-->

Commit message: Added new STL files and updated URDF files to match new rover model - still need to enter wheel separation data

File: description/rover_model/urdf/constants.xacro (robot description, xacro)
@@ -6,8 +6,8 @@
     <xacro:property name="base_height" value="0.01"/> -->
     <!-- Chassis -->
-    <xacro:property name="chassis_to_base_link_dist" value="0.34041"/>
-    <xacro:property name="chassis_to_stand_link_z_dist" value="0.26861"/>
-    <xacro:property name="chassis_to_stand_link_x_dist" value="0.178"/>
-    <xacro:property name="chassis_link_mass" value="36.95"/>
+    <xacro:property name="chassis_to_base_link_dist" value="0.428727"/>
+    <xacro:property name="chassis_to_stand_link_z_dist" value="0.354330"/>
+    <xacro:property name="chassis_to_stand_link_x_dist" value="0.3177"/>
+    <xacro:property name="chassis_link_mass" value="47.386726"/>
     <!-- Stand -->
     <!-- <xacro:property name="stand_length" value="0.412"/>
@@ -63,5 +63,5 @@
     <xacro:property name="top_laser_topicName" value="scan_upper"/>
     <xacro:property name="top_laser_frameName" value="top_lidar_link"/>
-    <xacro:property name="distance_to_second_lidar" value="0.14"/>
+    <xacro:property name="distance_to_second_lidar" value="0.13079"/>
     <!-- ZED camera -->
     <!-- NOTE: approx as a rectangular prism -->
@@ -90,5 +90,5 @@
     <!--ZED CAMERA JOINT PARAMETERS-->
     <xacro:property name="ZED_camera_to_top_plate_x" value="${(stand_width / 2.0)-0.01}"/>
-    <xacro:property name="ZED_camera_to_top_plate_z" value="0.10098"/>
+    <xacro:property name="ZED_camera_to_top_plate_z" value="0.085525"/>
     <!-- Garmin GPS -->
     <!-- NOTE: approx. as a cylinder, Garmin itself is similar to a hockey puck -->

File: description/rover_model/urdf/espresso.urdf.xacro (robot description, xacro)
@@ -14,14 +14,14 @@
 	<link name="chassis_link">
 		<inertial>
-			<origin xyz="-0.040859 0.00033673 -0.054592" rpy="0 0 0" />
-			<mass value="40.135" />
-			<inertia
-				ixx="0.58726"
-				ixy="1.3916E-05"
-				ixz="8.6833E-05"
-				iyy="0.27783"
-				iyz="1.0234E-06"
-				izz="0.67281" />
-		</inertial>
+			<origin xyz="0.099137 -0.018842 -0.136079" rpy="0 0 0" />
+            <mass value="47.386726" />
+            <inertia
+                ixx="1.885415"
+                ixy="-0.509416"
+                ixz="-0.934927"
+                iyy="5.617588"
+                iyz="0.116315"
+                izz="6.279312" />
+        </inertial>
 		<visual>
 			<origin xyz="0 0 0" rpy="0 0 0" />
@@ -41,5 +41,5 @@
 	</link>
 	<joint name="chassis_joint" type="fixed">
-		<origin xyz="0 0 0.34041" rpy="0 0 0" />
+		<origin xyz="0 0 0.428727" rpy="0 0 0" />
 		<parent link="base_link" />
 		<child link="chassis_link" />
@@ -52,5 +52,5 @@
 	<link name="top_lidar_link">
 		<inertial>
-			<origin xyz="0.012061 -0.00053309 -0.018931" rpy="0 0 0" />
+			<origin xyz="0.012061 0.0 -0.018931" rpy="0 0 0" />
 			<mass value="0.073082" />
 			<inertia
@@ -65,5 +65,5 @@
 			<origin xyz="0 0 0" rpy="0 0 0" />
 			<geometry>
-				<mesh filename="package://description/rover_model/meshes/lidar_link.STL" />
+				<mesh filename="package://description/rover_model/meshes/upper_lidar_link.STL" />
 			</geometry>
 			<material name="">
@@ -74,11 +74,11 @@
 			<origin xyz="0 0 0" rpy="0 0 0" />
 			<geometry>
-				<mesh filename="package://description/rover_model/meshes/lidar_link.STL" />
+				<mesh filename="package://description/rover_model/meshes/upper_lidar_link.STL" />
 			</geometry>
 		</collision>
 	</link>
 	<joint name="top_lidar_joint" type="fixed">
-		<origin xyz="0.52049 -0.005698 ${distance_to_second_lidar - 0.069334}" rpy="0 0 0" />
-		<!-- before z =  0.0056661 -->
+		<origin xyz="0.664824 0.0 ${distance_to_second_lidar - 0.185382}" rpy="0 0 0" />
+		<!--  -->
 		<parent link="chassis_link" />
 		<child link="top_lidar_link" />
@@ -91,5 +91,5 @@
 	<link name="bottom_lidar_link">
 		<inertial>
-			<origin xyz="-0.044335 2.8732E-05 -0.021084" rpy="0 0 0" />
+			<origin xyz="-0.044335 0.0 -0.021084" rpy="0 0 0" />
 			<mass value="0.46918" />
 			<inertia
@@ -118,5 +118,5 @@
 	</link>
 	<joint name="bottom_lidar_joint" type="fixed">
-		<origin xyz="0.52049 -0.005698 -0.069334" rpy="0 0 0" />
+		<origin xyz="0.664824 0.0 -0.185382" rpy="0 0 0" />
 		<parent link="chassis_link" />
 		<child link="bottom_lidar_link" />

File: description/rover_model/urdf/stand_link.urdf.xacro (robot description, xacro)
@@ -8,13 +8,13 @@
     <link name="stand_link">
         <inertial>
-            <origin xyz="0.000229157903262472 0.0038685225549956 0.00576901453025613" rpy="0 0 0" />
-            <mass value="0.230738007647473" />
+            <origin xyz="-0.003866 0.005769 0.000194" rpy="0 0 0" />
+            <mass value="0.327857" />
             <inertia
-                ixx="0.0007751891369661"
-                ixy="1.42155279926012E-07"
-                ixz="-1.93289911661184E-06"
-                iyy="0.000429374438189671"
-                iyz="1.9215645736234E-08"
-                izz="0.00119774793119647" />
+                ixx="0.000640"
+                ixy="-0.000013"
+                ixz="0.000055"
+                iyy="0.001837"
+                iyz=" -0.000004"
+                izz="0.001209" />
         </inertial>
         <visual>
@@ -35,5 +35,5 @@
     </link>
     <joint name="stand_joint" type="fixed">
-        <origin xyz="0.178 0.001524 0.26861" rpy="0 0 0" />
+        <origin xyz="0.3177 0.0 0.354330" rpy="0 0 0" />
         <parent link="chassis_link" />
         <child link="stand_link" />
@@ -74,5 +74,5 @@
     </link>
     <joint name="zed_joint" type="fixed">
-        <origin xyz="0.044163 0 ${ZED_camera_to_top_plate_z}" rpy="0 ${ZED_camera_pitch} 0" />
+        <origin xyz="0.0462 0 ${ZED_camera_to_top_plate_z}" rpy="0 ${ZED_camera_pitch} 0" />
         <parent link="stand_link" />
         <child link="zed_link" />
@@ -130,7 +130,8 @@
     </link>
     <joint name="imu_joint" type="fixed">
-        <origin xyz="0.159347 0 0" rpy="0 0 0" />
+        <origin xyz="0.275329 0 0.798932" rpy="0 0 0" />
         <!-- The x-pos is same as it's actual position on the stand, but z-pos same as base_link
              x: imu_x_dist_to_stand + chassis_to_stand_link_x_dist -->
+        <!-- delta x = 0.370205 ub reality -->
         <parent link="base_link" /> <!-- The frame origin is centered on base_link -->
         <child link="imu_link" />
@@ -170,5 +171,5 @@
     </link>
     <joint name="gps_joint" type="fixed">
-        <origin xyz="-0.054799 0 0.0095015" rpy="0 0 0" />
+        <origin xyz="-0.0502 0.062701 0.0095015" rpy="0 0 0" />
         <parent link="stand_link" />
         <child link="gps_link" />

File: description/rover_model/urdf/wheels.urdf.xacro (robot description, xacro)
@@ -17,5 +17,5 @@
     <link name="left_wheel_link">
         <inertial>
-            <origin xyz="-8.2128E-11 0 9.544E-08" rpy="0 0 0" />
+            <origin xyz="0.0 0.0 0.0" rpy="0 0 0" />
             <mass value="3.533" />
             <inertia
@@ -44,5 +44,5 @@
     </link>
     <joint name="left_wheel_joint" type="continuous">
-        <origin xyz="0.30478 0.40518 -0.21541" rpy="0 0 0" />
+        <origin xyz="0.390894 0.295916 -0.267008" rpy="0 0 0" />
         <parent link="chassis_link" />
         <child link="left_wheel_link" />
@@ -87,5 +87,5 @@
     </link>
     <joint name="right_wheel_joint" type="continuous">
-        <origin xyz="0.30482 -0.40518 -0.21541" rpy="0 0 0" />
+        <origin xyz="0.390894 -0.295916 -0.267008" rpy="0 0 0" />
         <parent link="chassis_link" />
         <child link="right_wheel_link" />
@@ -103,5 +103,5 @@
     <link name="caster_link">
         <inertial>
-            <origin xyz="-0.02078 3.2838E-05 -0.11441" rpy="0 0 0" />
+            <origin xyz="-0.02078 0.0 -0.11441" rpy="0 0 0" />
             <mass value="1.0439" />
             <inertia
@@ -130,5 +130,5 @@
     </link>
     <joint name="caster_joint" type="fixed">
-        <origin xyz="-0.36833 0.001524 -0.13183" rpy="0 0 0" />
+        <origin xyz="-0.222265 0.0 -0.212725" rpy="0 0 0" />
         <parent link="chassis_link" />
         <child link="caster_link" />

Commit message: Updated wheel separation distance

File: description/rover_model/urdf/constants.xacro (robot description, xacro)
@@ -26,5 +26,5 @@
     <xacro:property name="wheel_left_joint" value="left_wheel_joint"/>
     <xacro:property name="wheel_right_joint" value="right_wheel_joint"/>
-    <xacro:property name="wheels_separation" value="0.823976"/>
+    <xacro:property name="wheels_separation" value="0.591832"/>
     <xacro:property name="wheel_diameter" value="0.25"/>
     <xacro:property name="wheel_acceleration" value="1.0"/>

Commit message: 12 update rover urdf (#13)
* Added new STL files and updated URDF files to match new rover model - still need to enter wheel separation data

* Create launch_rover.sh

* Matching imu_denoiser.py to primary_laptop

* Fixing odom_global.yaml to only use odom local and gps

* Matching to primary_laptop

* Matchin to primary_laptop branch

* Matching to primary_laptop branch

* Adding packages for running wheel odom on laptop

* Updated wheel separation distance

* Add files via upload

Updated models of upper lidar and chassis_link for scaling.

---------

Co-authored-by: Ivy Tan <ivtn0912@gmail.com>
Co-authored-by: luotiger <114829395+luotiger@users.noreply.github.com>
Co-authored-by: tigrehomme <tigerluo03@gmail.com>
Co-authored-by: 1gaurg1 <121359236+1gaurg1@users.noreply.github.com>

File: description/rover_model/urdf/constants.xacro (robot description, xacro)
@@ -6,8 +6,8 @@
     <xacro:property name="base_height" value="0.01"/> -->
     <!-- Chassis -->
-    <xacro:property name="chassis_to_base_link_dist" value="0.34041"/>
-    <xacro:property name="chassis_to_stand_link_z_dist" value="0.26861"/>
-    <xacro:property name="chassis_to_stand_link_x_dist" value="0.178"/>
-    <xacro:property name="chassis_link_mass" value="36.95"/>
+    <xacro:property name="chassis_to_base_link_dist" value="0.428727"/>
+    <xacro:property name="chassis_to_stand_link_z_dist" value="0.354330"/>
+    <xacro:property name="chassis_to_stand_link_x_dist" value="0.3177"/>
+    <xacro:property name="chassis_link_mass" value="47.386726"/>
     <!-- Stand -->
     <!-- <xacro:property name="stand_length" value="0.412"/>
@@ -26,5 +26,5 @@
     <xacro:property name="wheel_left_joint" value="left_wheel_joint"/>
     <xacro:property name="wheel_right_joint" value="right_wheel_joint"/>
-    <xacro:property name="wheels_separation" value="0.823976"/>
+    <xacro:property name="wheels_separation" value="0.591832"/>
     <xacro:property name="wheel_diameter" value="0.25"/>
     <xacro:property name="wheel_acceleration" value="1.0"/>
@@ -63,5 +63,5 @@
     <xacro:property name="top_laser_topicName" value="scan_upper"/>
     <xacro:property name="top_laser_frameName" value="top_lidar_link"/>
-    <xacro:property name="distance_to_second_lidar" value="0.14"/>
+    <xacro:property name="distance_to_second_lidar" value="0.13079"/>
     <!-- ZED camera -->
     <!-- NOTE: approx as a rectangular prism -->
@@ -90,5 +90,5 @@
     <!--ZED CAMERA JOINT PARAMETERS-->
     <xacro:property name="ZED_camera_to_top_plate_x" value="${(stand_width / 2.0)-0.01}"/>
-    <xacro:property name="ZED_camera_to_top_plate_z" value="0.10098"/>
+    <xacro:property name="ZED_camera_to_top_plate_z" value="0.085525"/>
     <!-- Garmin GPS -->
     <!-- NOTE: approx. as a cylinder, Garmin itself is similar to a hockey puck -->
